File: examples/differential_hatched/differential.kicad_sch (KiCad schematic)
At the start: 5 parts

Commit message: Update examples with corrected settings and keep track of exported gerbers
Parts:
- GND1: footprint custom:test_pad_0 -> simulation_port:pad_0.05mm
- SP0, SP1, SP2, SP3: footprint custom:test_pad_0 -> simulation_port:pad_0.1mm
Changed lines of the file:
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@@
 			)
 		)
-		(property "Footprint" "custom:test_pad_0"
+		(property "Footprint" "simulation_port:pad_0.1mm"
 			(at 118.11 71.12 0)
 			(effects
@@
 			)
 		)
-		(property "Footprint" "custom:test_pad_0"
+		(property "Footprint" "simulation_port:pad_0.1mm"
 			(at 107.95 134.62 0)
 			(effects
@@
 			)
 		)
-		(property "Footprint" "custom:test_pad_0"
+		(property "Footprint" "simulation_port:pad_0.1mm"
 			(at 144.78 71.12 0)
 			(effects
@@
 			)
 		)
-		(property "Footprint" "custom:test_pad_0"
+		(property "Footprint" "simulation_port:pad_0.1mm"
 			(at 134.62 134.62 0)
 			(effects
@@
 			)
 		)
-		(property "Footprint" "custom:test_pad_0"
+		(property "Footprint" "simulation_port:pad_0.05mm"
 			(at 172.72 71.12 0)
 			(effects
